File: fuelguage.kicad_pcb (KiCad board)
At the start: 2 copper layers, 5 parts, among them IC1 LTC2941IMS8E#PBF

Commit message: prep for final
Parts:
- IC1: footprint Fuelguage ltc:SOP65P490X110-9N -> Library:SOP65P490X110-9N
- R1: footprint 2.2k:RESC2012X65N -> Library:RESC2012X65N
- R2, R3, R4: footprint RST 0.025:CRA2512-FZ-R025ELF -> Library:CRA2512-FZ-R025ELF
Changed lines of the file:
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@@
   (net 9 "unconnected-(IC1-EP-Pad9)")
   (net 10 "3.3V")
-  (footprint "RST 0.025:CRA2512-FZ-R025ELF" (layer "F.Cu")
+  (footprint "Library:CRA2512-FZ-R025ELF" (layer "F.Cu")
     (at 186.69 75.184 -90)
     (property "Sheetfile" "fuelguage.kicad_sch")
@@
     (pad "2" smd rect (at 2.9845 0 270) (size 1.397 3.5306) (layers "F.Cu" "F.Paste" "F.Mask")
       (net 6 "Net-(IC1-SDA)") (pintype "passive"))
-    (model "/mnt/DAA829C1A8299CCF/EEE/S7/PROJ/COMPS/RST/0.025/ul_CRA2512-FZ-R025ELF/2023-01-03_07-54-13/STEP/BO_CRA2512.step"
+    (model "${KIPRJMOD}/packages3D/BO_CRA2512.step"
       (offset (xyz 0 0 0))
       (scale (xyz 1 1 1))
@@
     )
   )
-  (footprint "Fuelguage ltc:SOP65P490X110-9N" (layer "F.Cu")
+  (footprint "Library:SOP65P490X110-9N" (layer "F.Cu")
     (at 171.524 76.241)
     (descr "MS8E Package 8-Lead Plastic MSOP, Exposed Die Pad")
@@
     (pad "9" smd rect (at 0 0) (size 1.68 1.88) (layers "F.Cu" "F.Paste" "F.Mask")
       (net 9 "unconnected-(IC1-EP-Pad9)") (pinfunction "EP") (pintype "passive"))
-    (model "LTC2941IMS8E#PBF.stp"
+    (model "${KIPRJMOD}/packages3D/LTC2941IMS8E#PBF.stp" hide
       (offset (xyz 0 0 0))
       (scale (xyz 1 1 1))
       (rotate (xyz 0 0 0))
     )
+    (model "${KIPRJMOD}/packages3D/LTC2941IMS8E#PBF.stp"
+      (offset (xyz 0 0 0))
+      (scale (xyz 1 1 1))
+      (rotate (xyz 0 0 0))
+    )
   )
-  (footprint "2.2k:RESC2012X65N" (layer "F.Cu")
+  (footprint "Library:RESC2012X65N" (layer "F.Cu")
     (at 171.704 72.644)
     (descr "SDR10")
@@
     (pad "2" smd rect (at 0.95 0) (size 1 1.4) (layers "F.Cu" "F.Paste" "F.Mask")
       (net 8 "Net-(IC1-SENSE-)") (pintype "passive"))
-    (model "SDR10EZPJ222.stp"
+    (model "${KIPRJMOD}/packages3D/SDR10EZPJ222.stp"
       (offset (xyz 0 0 0))
       (scale (xyz 1 1 1))
@@
     )
   )
-  (footprint "RST 0.025:CRA2512-FZ-R025ELF" (layer "F.Cu")
+  (footprint "Library:CRA2512-FZ-R025ELF" (layer "F.Cu")
     (at 164.592 73.7235 90)
     (property "Sheetfile" "fuelguage.kicad_sch")
@@
     (pad "2" smd rect (at 2.9845 0 90) (size 1.397 3.5306) (layers "F.Cu" "F.Paste" "F.Mask")
       (net 10 "3.3V") (pintype "passive"))
-    (model "/mnt/DAA829C1A8299CCF/EEE/S7/PROJ/COMPS/RST/0.025/ul_CRA2512-FZ-R025ELF/2023-01-03_07-54-13/STEP/BO_CRA2512.step"
+    (model "${KIPRJMOD}/packages3D/BO_CRA2512.step"
       (offset (xyz 0 0 0))
       (scale (xyz 1 1 1))
@@
     )
   )
-  (footprint "RST 0.025:CRA2512-FZ-R025ELF" (layer "F.Cu")
+  (footprint "Library:CRA2512-FZ-R025ELF" (layer "F.Cu")
     (at 179.07 72.39 -90)
     (property "Sheetfile" "fuelguage.kicad_sch")
@@
     (pad "2" smd rect (at 2.9845 0 270) (size 1.397 3.5306) (layers "F.Cu" "F.Paste" "F.Mask")
       (net 7 "Net-(IC1-~{AL}{slash}CC)") (pintype "passive"))
-    (model "/mnt/DAA829C1A8299CCF/EEE/S7/PROJ/COMPS/RST/0.025/ul_CRA2512-FZ-R025ELF/2023-01-03_07-54-13/STEP/BO_CRA2512.step"
+    (model "${KIPRJMOD}/packages3D/BO_CRA2512.step"
       (offset (xyz 0 0 0))
       (scale (xyz 1 1 1))
